File: bcd_schematics/9thbutton.kicad_sch (KiCad schematic)
At the start: 27 parts, among them SW1 1, SW2 2, SW3 3, SW4 4, SW5 5, SW6 6, SW7 7, SW8 8, SW9 9, U1 4072, U2 4072

Commit message: 9th Button Schematics
Parts:
- added 10K: R, symbol Device:R
- added OR 1: 74LS32, symbol 74xx:74LS32
- renumbered R13 to 10K, R5 to 10K, R3 to 10K, R2 to 10K, R14 to 10K, R6 to 10K, R16 to 10K, R12 to 10K, R11 to 10K, R4 to 10K, R1 to 10K, R10 to 10K, R9 to 10K, R8 to 10K, R15 to 10K, R7 to 10K
Connections:
- net GND: now also 10K.2
- net at 10K.1, U2.10: now also SW9.2, 10K.1, OR 1.2
- net at 10K.1, 10K.1, 10K.1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: now also OR 1.1; no longer U2.5
- net 1 renamed D1
- net 2 renamed D2
- net 3 renamed D3
- net 4 renamed D4
- new net: OR 1.3, U2.5
Other:
- moved on the sheet: 10K, SW1, SW2, SW3, SW4, SW5, SW6, SW7, SW8, SW9, U1A, U1B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
